File: board/MiniSSO/MiniSSO.kicad_pcb (KiCad board)
At the start: 2 copper layers, 50.8 x 22.9 mm, 36 parts, among them J1 Conn_01x02, J2 Conn_01x02, J3 Conn_01x16, J4 Conn_01x03, J5 Conn_01x12, Q1 MCU30N02-TP, Q2 MCU30N02-TP, SW1 SW_Push, U2 LTV-356T

Commit message: Rev 1: Initial version of the board.
Parts:
- removed R1: 560, Resistor_SMD:R_0603_1608Metric
- D4, D6: value D_Schottky -> SBA130AS_R1_00001
- R11: value 220 -> 470
- R12: value 150 -> 1k
- R2, R5: value R -> 68
- moved G*** 17.9 mm to (148.5, 77.3)
Connections:
- U2 pad 2: Net-(R1-Pad1) -> Net-(D1-Pad2)
Routing:
- net Net-(D1-Pad2): track 1.54 -> 7.59 mm
- net Net-(R1-Pad1): track 4.41 -> 0.00 mm
Other:
- board text added: "+"
- board text added: "-"
- board text added: "1"
- board text added: "2"
- board text added: "MiniSSO"
- board text added: "MiniSSO 2 1.5A 12V Dimmable Outputs 1 12V Isolated Trigger Input"
- board text added: "Out 1"
- board text added: "Out 1 TP"
- board text added: "Out 2"
- board text added: "Out 2 TP"
- board text added: "Output"
- board text added: "Output 2"
- board text added: "Rev 1"
- board text added: "Trig"
- board text removed: "ESP32-S2 MiniMain 240MHz Tensilica WiFi 4 MByte FLASH 2 MByte PSRAM"
