File: board/MiniSSO/MiniSSO.kicad_sch (KiCad schematic)
At the start: 35 parts, among them J1 Conn_01x02, J2 Conn_01x02, J3 Conn_01x16, J4 Conn_01x03, J5 Conn_01x12, Q1 MCU30N02-TP, Q2 MCU30N02-TP, SW1 SW_Push, U2 LTV-356T

Commit message: Rev 1: Initial version of the board.
Parts:
- removed R1: 560, Resistor_SMD:R_0603_1608Metric, symbol Device:R
- D4, D6: value D_Schottky -> SBA130AS_R1_00001
- R11: value 220 -> 470
- R12: value 150 -> 1k
- R2, R5: value R -> 68
Connections:
- net GND: no longer H1.1, H3.1
- net at U2.2: now also D1.2 (A)
- new net: H1.1, H3.1
Other:
- note added: "691214110002 ALT YO0201500000G"
- note added: "691214110003 ALT EBWA-03-A"
- note added: "ALT 1N4148W-AU_R1_000A1"
- note removed: "691214110002"
- note removed: "691214110003"
- company: (none) -> Department of Alchemy
- title: (none) -> MiniSSO
- moved on the sheet: H1, H2, H3, H4
